Commit message: urdf file finished and ready to vis with rviz

File: urdf/barista_robot_model.urdf (robot description, URDF)
Before this commit: robot box_bot, 10 links, 9 joints
Links:
- added link back_left_pillar; visual cylinder length=0.22 radius=0.01
- added link back_right_pillar; visual cylinder length=0.22 radius=0.01
- added link cup_holder; visual cylinder length=0.09 radius=0.17
- added link front_left_pillar; visual cylinder length=0.22 radius=0.01
- added link front_right_pillar; visual cylinder length=0.22 radius=0.01
Joints:
- added joint back_left_pillar_joint: type fixed, parent base_link, child back_left_pillar, origin xyz=-0.025 0.15 0.1875 rpy=0 0 0
- added joint back_right_pillar_joint: type fixed, parent base_link, child back_right_pillar, origin xyz=-0.025 -0.15 0.1875 rpy=0 0 0
- added joint cup_holder_joint: type fixed, parent base_link, child cup_holder, origin xyz=0.0 0.0 0.3425 rpy=0 0 0
- added joint front_left_pillar_joint: type fixed, parent base_link, child front_left_pillar, origin xyz=0.025 0.15 0.1875 rpy=0 0 0
- added joint front_right_pillar_joint: type fixed, parent base_link, child front_right_pillar, origin xyz=0.025 -0.15 0.1875 rpy=0 0 0
- joint back_yaw_joint: origin xyz=-0.1 0 -0.0775 rpy=0 0 0 -> xyz=-0.12 0 -0.1 rpy=0 0 0
- joint front_yaw_joint: origin xyz=0.1 0 -0.0775 rpy=0 0 0 -> xyz=0.12 0 -0.1 rpy=0 0 0
- joint joint_left_wheel: origin xyz=0 0.1 -0.0775 rpy=0 0 0 -> xyz=0 0.12 -0.0775 rpy=0 0 0
- joint joint_right_wheel: origin xyz=0 -0.1 -0.0775 rpy=0 0 0 -> xyz=0 -0.12 -0.0775 rpy=0 0 0

Commit message: launch files for gazebbo test add, collisions and mass ad to each part of robot

File: urdf/barista_robot_model.urdf (robot description, URDF)
Before this commit: robot box_bot, 15 links, 14 joints
Links:
- link back_left_pillar: mass None -> 0.42857142857142855; geometry collision cylinder length=0.22 radius=0.01; visual cylinder length=0.22 radius=0.01
- link back_right_pillar: mass None -> 0.42857142857142855; geometry collision cylinder length=0.22 radius=0.01; visual cylinder length=0.22 radius=0.01
- link back_yaw_link: mass None -> 0.42857142857142855; geometry collision cylinder length=0.005 radius=0.010; visual cylinder length=0.005 radius=0.010
- link chassis: mass None -> 0.42857142857142855; geometry collision cylinder length=0.155 radius=0.178; visual cylinder length=0.155 radius=0.178
- link cup_holder: mass None -> 0.42857142857142855; geometry collision cylinder length=0.22 radius=0.01; visual cylinder length=0.09 radius=0.17
- link front_left_pillar: mass None -> 0.42857142857142855; geometry collision cylinder length=0.22 radius=0.01; visual cylinder length=0.22 radius=0.01
- link front_right_pillar: mass None -> 0.42857142857142855; geometry collision cylinder length=0.22 radius=0.01; visual cylinder length=0.22 radius=0.01
- link front_yaw_link: mass None -> 0.42857142857142855; geometry collision cylinder length=0.005 radius=0.010; visual cylinder length=0.005 radius=0.010
- link left_wheel: mass None -> 0.42857142857142855; geometry collision cylinder length=0.0206 radius=0.0352; visual cylinder length=0.0206 radius=0.0352
- link right_wheel: mass None -> 0.42857142857142855; geometry collision cylinder length=0.0206 radius=0.0352; visual cylinder length=0.0206 radius=0.0352

Commit message: robot ready for sensor install, gazebo launch options added

File: urdf/barista_robot_model.urdf (robot description, URDF)
Before this commit: robot box_bot, 15 links, 14 joints
Links:
- added link lidar; visual mesh filename=package://barista_robot_description/meshes/hokuyo_urg_04lx.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
- link back_pitch_link: mass None -> 0.001; geometry collision cylinder length=0.001 radius=0.0045000000000000005; visual cylinder length=0.001 radius=0.0045000000000000005
- link back_roll_link: mass None -> 0.001; geometry collision cylinder length=0.001 radius=0.0045000000000000005; visual cylinder length=0.001 radius=0.0045000000000000005
- link back_yaw_link: mass 0.42857142857142855 -> 0.001; geometry collision cylinder length=0.001 radius=0.0045000000000000005; visual cylinder length=0.001 radius=0.0045000000000000005
- link cup_holder: geometry collision cylinder length=0.09 radius=0.17; visual cylinder length=0.09 radius=0.17
- link front_pitch_link: mass None -> 0.001; geometry collision cylinder length=0.001 radius=0.0045000000000000005; visual cylinder length=0.001 radius=0.0045000000000000005
- link front_roll_link: mass None -> 0.001; geometry collision cylinder length=0.001 radius=0.0045000000000000005; visual cylinder length=0.001 radius=0.0045000000000000005
- link front_yaw_link: mass 0.42857142857142855 -> 0.001; geometry collision cylinder length=0.001 radius=0.0045000000000000005; visual cylinder length=0.001 radius=0.0045000000000000005
Joints:
- added joint lidar_joint: type fixed, parent base_link, child lidar, origin xyz=-0.05 0 0.0775 rpy=0 0 0
- joint back_yaw_joint: origin xyz=-0.12 0 -0.1 rpy=0 0 0 -> xyz=-0.12 0 -0.1082 rpy=0 0 0
- joint front_yaw_joint: origin xyz=0.12 0 -0.1 rpy=0 0 0 -> xyz=0.12 0 -0.1082 rpy=0 0 0

Commit message: laser plugin add, ready to xacrofy

File: urdf/barista_robot_model.urdf (robot description, URDF)
Before this commit: robot box_bot, 16 links, 15 joints
Joints:
- joint lidar_joint: origin xyz=-0.05 0 0.0775 rpy=0 0 0 -> xyz=-0.05 0 0.125 rpy=0 0 0
