Commit message: xacro file modified to spawn two robots

File: xacro/barista_robot_model.urdf.xacro (robot description, xacro)
@@ -8,8 +8,10 @@
 <!-- Define the argument for including the laser -->
 <xacro:arg name="include_laser" default="true" />
+<xacro:arg name="robot_name" default="barista" />
+<xacro:property name="robot_name_prop" value="$(arg robot_name)"/>
 <!-- Lidar Sensor Macro Definition -->
 <xacro:macro name="laser_scanner">
     <!-- Lidar Sensor -->
-    <link name="lidar">
+    <link name="${robot_name_prop}_lidar">
         <visual>
             <origin rpy="0 0 0" xyz="0.0 0 -0.05" />
@@ -19,14 +21,12 @@
         </visual>
     </link>
-    <joint name="lidar_joint" type="fixed">
+    <joint name="${robot_name_prop}_lidar_joint" type="fixed">
         <origin rpy="0 0 0" xyz="-0.05 0 0.125" />
-        <parent link="base_link" />
-        <child link="lidar" />
+        <parent link="${robot_name_prop}_base_link" />
+        <child link="${robot_name_prop}_lidar" />
     </joint>
+    <!-- Lidar plugin -->
     <gazebo reference="lidar">
         <material>Gazebo/Black</material>
-    </gazebo>
-    <!-- Lidar plugin -->
-    <gazebo reference="lidar">
         <sensor name="sensor_ray" type="ray">
             <pose>0 0 0 0 0 0</pose>
@@ -48,7 +48,7 @@
             <visualize>true</visualize>
             <update_rate>100.0</update_rate>
-            <plugin name="laser" filename="libgazebo_ros_ray_sensor.so">
+            <plugin name="${robot_name_prop}_laser" filename="libgazebo_ros_ray_sensor.so">
                 <ros>
-                    <remapping>~/out:=scan</remapping>
+                    <remapping>~/out:=/${robot_name_prop}/scan</remapping>
                 </ros>
                 <output_type>sensor_msgs/LaserScan</output_type>
@@ -73,8 +73,8 @@
     <color rgba="0.088656 0.428691 0.491021 1" />
   </material>
-  <link name="base_link">
+  <link name="${robot_name_prop}_base_link">
   </link>
   <!-- Body -->
-  <link name="chassis">
+  <link name="${robot_name_prop}_chassis">
     <visual>
       <geometry>
@@ -94,51 +94,51 @@
     </inertial>
   </link>
-  <joint name="base_link_joint" type="fixed">
+  <joint name="${robot_name_prop}_base_link_joint" type="fixed">
     <origin rpy="0 0 0" xyz="0 0 0" />
-    <parent link="base_link" />
-    <child link="chassis" />
-  </joint>
-  <gazebo reference="chassis">
+    <parent link="${robot_name_prop}_base_link" />
+    <child link="${robot_name_prop}_chassis" />
+  </joint>
+  <gazebo reference="${robot_name_prop}_chassis">
         <material>Gazebo/Blue</material>
   </gazebo>
   <!-- Front standoffs -->
-  <xacro:standoff name="front_right_standoff" />
-  <joint name="front_right_standoff_joint" type="fixed">
+  <xacro:standoff name="${robot_name_prop}_front_right_standoff" />
+  <joint name="${robot_name_prop}_front_right_standoff_joint" type="fixed">
     <origin rpy="0 0 0" xyz="0.025 -0.15 0.1875" />
-    <parent link="base_link" />
-    <child link="front_right_standoff" />
-  </joint>
-  <xacro:standoff name="front_left_standoff" />
-  <joint name="front_left_standoff_joint" type="fixed">
+    <parent link="${robot_name_prop}_base_link" />
+    <child link="${robot_name_prop}_front_right_standoff" />
+  </joint>
+  <xacro:standoff name="${robot_name_prop}_front_left_standoff" />
+  <joint name="${robot_name_prop}_front_left_standoff_joint" type="fixed">
     <origin rpy="0 0 0" xyz="0.025 0.15 0.1875" />
-    <parent link="base_link" />
-    <child link="front_left_standoff" />
+    <parent link="${robot_name_prop}_base_link" />
+    <child link="${robot_name_prop}_front_left_standoff" />
   </joint>
   <!-- Back standoffs -->
-  <xacro:standoff name="back_right_standoff" />
-  <joint name="back_right_standoff_joint" type="fixed">
+  <xacro:standoff name="${robot_name_prop}_back_right_standoff" />
+  <joint name="${robot_name_prop}_back_right_standoff_joint" type="fixed">
     <origin rpy="0 0 0" xyz="-0.025 -0.15 0.1875" />
-    <parent link="base_link" />
-    <child link="back_right_standoff" />
-  </joint>
-  <xacro:standoff name="back_left_standoff" />
-  <joint name="back_left_standoff_joint" type="fixed">
+    <parent link="${robot_name_prop}_base_link" />
+    <child link="${robot_name_prop}_back_right_standoff" />
+  </joint>
+  <xacro:standoff name="${robot_name_prop}_back_left_standoff" />
+  <joint name="${robot_name_prop}_back_left_standoff_joint" type="fixed">
     <origin rpy="0 0 0" xyz="-0.025 0.15 0.1875" />
-    <parent link="base_link" />
-    <child link="back_left_standoff" />
+    <parent link="${robot_name_prop}_base_link" />
+    <child link="${robot_name_prop}_back_left_standoff" />
   </joint>
   <!-- Cup holder tray -->
-  <xacro:cup_holder_tray name="cup_holder" />
-  <joint name="cup_holder_joint" type="fixed">
+  <xacro:cup_holder_tray name="${robot_name_prop}_cup_holder" />
+  <joint name="${robot_name_prop}_cup_holder_joint" type="fixed">
     <origin rpy="0 0 0" xyz="0.0 0.0 0.3425" />
-    <parent link="base_link" />
-    <child link="cup_holder" />
-  </joint>
-  <gazebo reference="cup_holder">
+    <parent link="${robot_name_prop}_base_link" />
+    <child link="${robot_name_prop}_cup_holder" />
+  </joint>
+  <gazebo reference="${robot_name_prop}_cup_holder">
         <material>Gazebo/Blue</material>
   </gazebo>
   <!-- Wheel Left -->
-  <xacro:wheel prefix="left" />
-  <gazebo reference="left_wheel">
+  <xacro:wheel prefix="${robot_name_prop}_left" />
+  <gazebo reference="${robot_name_prop}_left_wheel">
     <kp>1000000000000000000000000000.0</kp>
     <kd>1000000000000000000000000000.0</kd>
@@ -147,8 +147,8 @@
     <material>Gazebo/Black</material>
   </gazebo>
-  <joint name="joint_left_wheel" type="continuous">
+  <joint name="${robot_name_prop}_joint_left_wheel" type="continuous">
     <origin rpy="0 0 0" xyz="0 0.12 -0.0775" />
-    <child link="left_wheel" />
-    <parent link="chassis" />
+    <child link="${robot_name_prop}_left_wheel" />
+    <parent link="${robot_name_prop}_chassis" />
     <axis rpy="0 0 0" xyz="0 1 0" />
     <limit effort="10000" velocity="1000" />
@@ -156,6 +156,6 @@
   </joint>
   <!-- Wheel Right -->
-  <xacro:wheel prefix="right" />
-  <gazebo reference="right_wheel">
+  <xacro:wheel prefix="${robot_name_prop}_right" />
+  <gazebo reference="${robot_name_prop}_right_wheel">
     <kp>1000000000000000000000000000.0</kp>
     <kd>1000000000000000000000000000.0</kd>
@@ -164,8 +164,8 @@
     <material>Gazebo/Black</material>
   </gazebo>
-  <joint name="joint_right_wheel" type="continuous">
+  <joint name="${robot_name_prop}_joint_right_wheel" type="continuous">
     <origin rpy="0 0 0" xyz="0 -0.12 -0.0775" />
-    <child link="right_wheel" />
-    <parent link="chassis" />
+    <child link="${robot_name_prop}_right_wheel" />
+    <parent link="${robot_name_prop}_chassis" />
     <axis rpy="0 0 0" xyz="0 1 0" />
     <limit effort="10000" velocity="1000" />
@@ -173,5 +173,5 @@
   </joint>
   <!-- Caster Wheel Front -->
-  <link name="front_yaw_link">
+  <link name="${robot_name_prop}_front_yaw_link">
     <visual>
       <origin rpy="0 1.5707 1.5707" xyz="0 0 0" />
@@ -193,16 +193,16 @@
     </inertial>
   </link>
-  <gazebo reference="front_yaw_link">
+  <gazebo reference="${robot_name_prop}_front_yaw_link">
         <material>Gazebo/Blue</material>
   </gazebo>
-  <joint name="front_yaw_joint" type="continuous">
+  <joint name="${robot_name_prop}_front_yaw_joint" type="continuous">
     <origin rpy="0 0 0" xyz="0.12 0 -0.1082" />
-    <parent link="chassis" />
-    <child link="front_yaw_link" />
+    <parent link="${robot_name_prop}_chassis" />
+    <child link="${robot_name_prop}_front_yaw_link" />
     <axis xyz="0 0 1" />
     <limit effort="1000.0" velocity="100.0" />
     <dynamics damping="0.0" friction="0.1" />
   </joint>
-  <link name="front_roll_link">
+  <link name="${robot_name_prop}_front_roll_link">
      <visual>
       <origin rpy="0 1.5707 1.5707" xyz="0 0 0" />
@@ -224,16 +224,16 @@
     </inertial>
   </link>
-  <gazebo reference="front_roll_link">
+  <gazebo reference="${robot_name_prop}_front_roll_link">
         <material>Gazebo/Red</material>
   </gazebo>
-  <joint name="front_roll_joint" type="continuous">
+  <joint name="${robot_name_prop}_front_roll_joint" type="continuous">
     <origin rpy="0 0 0" xyz="0 0 0" />
-    <parent link="front_yaw_link" />
-    <child link="front_roll_link" />
+    <parent link="${robot_name_prop}_front_yaw_link" />
+    <child link="${robot_name_prop}_front_roll_link" />
     <axis xyz="1 0 0" />
     <limit effort="1000.0" velocity="100.0" />
     <dynamics damping="0.0" friction="0.1" />
   </joint>
-  <link name="front_pitch_link">
+  <link name="${robot_name_prop}_front_pitch_link">
      <visual>
       <origin rpy="0 1.5707 1.5707" xyz="0 0 0" />
@@ -255,5 +255,5 @@
     </inertial>
   </link>
-  <gazebo reference="front_pitch_link">
+  <gazebo reference="${robot_name_prop}_front_pitch_link">
     <kp>1000000000000000000000000000.0</kp>
     <kd>1000000000000000000000000000.0</kd>
@@ -262,8 +262,8 @@
     <material>Gazebo/Purple</material>
   </gazebo>
-  <joint name="front_pitch_joint" type="continuous">
+  <joint name="${robot_name_prop}_front_pitch_joint" type="continuous">
     <origin rpy="0 0 0" xyz="0 0 0" />
-    <parent link="front_roll_link" />
-    <child link="front_pitch_link" />
+    <parent link="${robot_name_prop}_front_roll_link" />
+    <child link="${robot_name_prop}_front_pitch_link" />
     <axis xyz="0 1 0" />
     <limit effort="1000.0" velocity="100.0" />
@@ -271,5 +271,5 @@
   </joint>
   <!-- Caster Wheel Back -->
-  <link name="back_yaw_link">
+  <link name="${robot_name_prop}_back_yaw_link">
      <visual>
       <origin rpy="0 1.5707 1.5707" xyz="0 0 0" />
@@ -291,16 +291,16 @@
     </inertial>
   </link>
-  <gazebo reference="back_yaw_link">
+  <gazebo reference="${robot_name_prop}_back_yaw_link">
         <material>Gazebo/Blue</material>
   </gazebo>
-  <joint name="back_yaw_joint" type="continuous">
+  <joint name="${robot_name_prop}_back_yaw_joint" type="continuous">
     <origin rpy="0 0 0" xyz="-0.12 0 -0.1082" />
-    <parent link="chassis" />
-    <child link="back_yaw_link" />
+    <parent link="${robot_name_prop}_chassis" />
+    <child link="${robot_name_prop}_back_yaw_link" />
     <axis xyz="0 0 1" />
     <limit effort="1000.0" velocity="100.0" />
     <dynamics damping="0.0" friction="0.1" />
   </joint>
-  <link name="back_roll_link">
+  <link name="${robot_name_prop}_back_roll_link">
      <visual>
       <origin rpy="0 1.5707 1.5707" xyz="0 0 0" />
@@ -322,16 +322,16 @@
     </inertial>
   </link>
-  <gazebo reference="back_roll_link">
+  <gazebo reference="${robot_name_prop}_back_roll_link">
         <material>Gazebo/Red</material>
   </gazebo>
-  <joint name="back_roll_joint" type="continuous">
+  <joint name="${robot_name_prop}_back_roll_joint" type="continuous">
     <origin rpy="0 0 0" xyz="0 0 0" />
-    <parent link="back_yaw_link" />
-    <child link="back_roll_link" />
+    <parent link="${robot_name_prop}_back_yaw_link" />
+    <child link="${robot_name_prop}_back_roll_link" />
     <axis xyz="1 0 0" />
     <limit effort="1000.0" velocity="100.0" />
     <dynamics damping="0.0" friction="0.1" />
   </joint>
-  <link name="back_pitch_link">
+  <link name="${robot_name_prop}_back_pitch_link">
      <visual>
       <origin rpy="0 1.5707 1.5707" xyz="0 0 0" />
@@ -353,5 +353,5 @@
     </inertial>
   </link>
-  <gazebo reference="back_pitch_link">
+  <gazebo reference="${robot_name_prop}_back_pitch_link">
     <kp>1000000000000000000000000000.0</kp>
     <kd>1000000000000000000000000000.0</kd>
@@ -360,8 +360,8 @@
     <material>Gazebo/Yellow</material>
   </gazebo>
-  <joint name="back_pitch_joint" type="continuous">
+  <joint name="${robot_name_prop}_back_pitch_joint" type="continuous">
     <origin rpy="0 0 0" xyz="0 0 0" />
-    <parent link="back_roll_link" />
-    <child link="back_pitch_link" />
+    <parent link="${robot_name_prop}_back_roll_link" />
+    <child link="${robot_name_prop}_back_pitch_link" />
     <axis xyz="0 1 0" />
     <limit effort="1000.0" velocity="100.0" />
@@ -371,25 +371,25 @@
   <!-- JOINT PUBLISHER -->
   <gazebo>
-    <plugin name="barista_robot_joint_state" filename="libgazebo_ros_joint_state_publisher.so">
+    <plugin name="${robot_name_prop}_robot_joint_state" filename="libgazebo_ros_joint_state_publisher.so">
       <ros>
-          <remapping>~/out:=joint_states</remapping>
+          <remapping>~/out:=/${robot_name_prop}/joint_states</remapping>
       </ros>
       <update_rate>30</update_rate>
-      <joint_name>joint_left_wheel</joint_name>
-      <joint_name>joint_right_wheel</joint_name>
-      <joint_name>front_yaw_joint</joint_name>
-      <joint_name>back_yaw_joint</joint_name>
-      <joint_name>front_roll_joint</joint_name>
-      <joint_name>back_roll_joint</joint_name>
-      <joint_name>front_pitch_joint</joint_name>
-      <joint_name>back_pitch_joint</joint_name>
+      <joint_name>${robot_name_prop}_joint_left_wheel</joint_name>
+      <joint_name>${robot_name_prop}_joint_right_wheel</joint_name>
+      <joint_name>${robot_name_prop}_front_yaw_joint</joint_name>
+      <joint_name>${robot_name_prop}_back_yaw_joint</joint_name>
+      <joint_name>${robot_name_prop}_front_roll_joint</joint_name>
+      <joint_name>${robot_name_prop}_back_roll_joint</joint_name>
+      <joint_name>${robot_name_prop}_front_pitch_joint</joint_name>
+      <joint_name>${robot_name_prop}_back_pitch_joint</joint_name>
     </plugin>
   </gazebo>
   <!-- Differential drive -->
   <gazebo>
-    <plugin filename="libgazebo_ros_diff_drive.so" name="differential_drive_controller">
+    <plugin filename="libgazebo_ros_diff_drive.so" name="{robot_name_prop}_differential_drive_controller">
       <!-- wheels -->
-      <left_joint>joint_left_wheel</left_joint>
-      <right_joint>joint_right_wheel</right_joint>
+      <left_joint>${robot_name_prop}_joint_left_wheel</left_joint>
+      <right_joint>${robot_name_prop}_joint_right_wheel</right_joint>
       <!-- kinematics -->
       <wheel_separation>0.24</wheel_separation>
@@ -401,6 +401,6 @@
       <publish_odom>true</publish_odom>
       <publish_odom_tf>true</publish_odom_tf>
-      <odometry_frame>odom</odometry_frame>
-      <robot_base_frame>base_link</robot_base_frame>
+      <odometry_frame>/${robot_name_prop}/odom</odometry_frame>
+      <robot_base_frame>${robot_name_prop}_base_link</robot_base_frame>
     </plugin>
   </gazebo>

Commit message: colors fixed

File: xacro/barista_robot_model.urdf.xacro (robot description, xacro)
@@ -10,4 +10,13 @@
 <xacro:arg name="robot_name" default="barista" />
 <xacro:property name="robot_name_prop" value="$(arg robot_name)"/>
+<xacro:property name="chassis_material" value="Gazebo/Blue"/>
+<!-- Check if the robot is Rick and set color to Blue -->
+<xacro:if value="${robot_name_prop == 'rick'}">
+  <xacro:property name="chassis_material" value="Gazebo/Blue"/>
+</xacro:if>
+<!-- Check if the robot is Morty and set color to Red -->
+<xacro:if value="${robot_name_prop == 'morty'}">
+  <xacro:property name="chassis_material" value="Gazebo/Red"/>
+</xacro:if>
 <!-- Lidar Sensor Macro Definition -->
 <xacro:macro name="laser_scanner">
@@ -100,5 +109,5 @@
   </joint>
   <gazebo reference="${robot_name_prop}_chassis">
-        <material>Gazebo/Blue</material>
+      <material>${chassis_material}</material>
   </gazebo>
   <!-- Front standoffs -->
@@ -136,5 +145,5 @@
   </joint>
   <gazebo reference="${robot_name_prop}_cup_holder">
-        <material>Gazebo/Blue</material>
+       <material>${chassis_material}</material>
   </gazebo>
   <!-- Wheel Left -->
