Commit message: issues with tf in rviz fixed, double joint publisher deleted, rviz color should be fixed

File: xacro/barista_robot_model.urdf.xacro (robot description, xacro)
@@ -9,12 +9,15 @@
 <xacro:arg name="include_laser" default="true" />
 <xacro:arg name="robot_name" default="barista" />
-<xacro:property name="robot_name_prop" value="$(arg robot_name)"/>
+<xacro:property name="robot_name" value="$(arg robot_name)"/>
 <xacro:property name="chassis_material" value="Gazebo/Blue"/>
+<xacro:property name="rviz_chassis_material_blue" value="blue"/>
+<xacro:property name="rviz_chassis_material_red" value="red"/>
 <!-- Check if the robot is Rick and set color to Blue -->
-<xacro:if value="${robot_name_prop == 'rick'}">
+<xacro:if value="${robot_name == 'rick'}">
   <xacro:property name="chassis_material" value="Gazebo/Blue"/>
+  <xacro:property name="rviz_material" value="${rviz_chassis_material_blue}"/>
 </xacro:if>
 <!-- Check if the robot is Morty and set color to Red -->
-<xacro:if value="${robot_name_prop == 'morty'}">
+<xacro:if value="${robot_name == 'morty'}">
   <xacro:property name="chassis_material" value="Gazebo/Red"/>
 </xacro:if>
@@ -22,5 +25,5 @@
 <xacro:macro name="laser_scanner">
     <!-- Lidar Sensor -->
-    <link name="${robot_name_prop}_lidar">
+    <link name="lidar">
         <visual>
             <origin rpy="0 0 0" xyz="0.0 0 -0.05" />
@@ -30,11 +33,11 @@
         </visual>
     </link>
-    <joint name="${robot_name_prop}_lidar_joint" type="fixed">
+    <joint name="lidar_joint" type="fixed">
         <origin rpy="0 0 0" xyz="-0.05 0 0.125" />
-        <parent link="${robot_name_prop}_base_link" />
-        <child link="${robot_name_prop}_lidar" />
+        <parent link="chassis" />
+        <child link="lidar" />
     </joint>
     <!-- Lidar plugin -->
-    <gazebo reference="${robot_name_prop}_lidar">
+    <gazebo reference="lidar">
         <material>Gazebo/Black</material>
         <sensor name="sensor_ray" type="ray">
@@ -57,8 +60,10 @@
             <visualize>true</visualize>
             <update_rate>100.0</update_rate>
-            <plugin name="${robot_name_prop}_laser" filename="libgazebo_ros_ray_sensor.so">
+            <plugin name="laser" filename="libgazebo_ros_ray_sensor.so">
                 <ros>
-                    <remapping>~/out:=/${robot_name_prop}/scan</remapping>
+                    <namespace>${robot_name}</namespace>
+                    <remapping>~/out:=/scan</remapping>
                 </ros>
+                <frame_name>${robot_name}/base_link</frame_name>
                 <output_type>sensor_msgs/LaserScan</output_type>
             </plugin>
@@ -70,7 +75,4 @@
     <xacro:laser_scanner />
 </xacro:if>
-  <material name="blue">
-    <color rgba="0.0 0.0 1.0 1" />
-  </material>
   <material name="black">
     <color rgba="0.0 0.0 0.0 1" />
@@ -82,13 +84,13 @@
     <color rgba="0.088656 0.428691 0.491021 1" />
   </material>
-  <link name="${robot_name_prop}_base_link">
+  <link name="base_link">
   </link>
   <!-- Body -->
-  <link name="${robot_name_prop}_chassis">
+  <link name="chassis">
     <visual>
       <geometry>
         <cylinder length="0.155" radius="0.178" />
       </geometry>
-      <material name="blue" />
+      <material name="rviz_material" />
     </visual>
     <collision>
@@ -103,61 +105,61 @@
     </inertial>
   </link>
-  <joint name="${robot_name_prop}_base_link_joint" type="fixed">
+  <joint name="base_link_joint" type="fixed">
     <origin rpy="0 0 0" xyz="0 0 0" />
-    <parent link="${robot_name_prop}_base_link" />
-    <child link="${robot_name_prop}_chassis" />
-  </joint>
-  <gazebo reference="${robot_name_prop}_chassis">
+    <parent link="base_link" />
+    <child link="chassis" />
+  </joint>
+  <gazebo reference="chassis">
       <material>${chassis_material}</material>
   </gazebo>
   <!-- Front standoffs -->
-  <xacro:standoff name="${robot_name_prop}_front_right_standoff" />
-  <joint name="${robot_name_prop}_front_right_standoff_joint" type="fixed">
+  <xacro:standoff name="front_right_standoff" />
+  <joint name="front_right_standoff_joint" type="fixed">
     <origin rpy="0 0 0" xyz="0.025 -0.15 0.1875" />
-    <parent link="${robot_name_prop}_base_link" />
-    <child link="${robot_name_prop}_front_right_standoff" />
-  </joint>
-  <xacro:standoff name="${robot_name_prop}_front_left_standoff" />
-  <joint name="${robot_name_prop}_front_left_standoff_joint" type="fixed">
+    <parent link="chassis" />
+    <child link="front_right_standoff" />
+  </joint>
+  <xacro:standoff name="front_left_standoff" />
+  <joint name="front_left_standoff_joint" type="fixed">
     <origin rpy="0 0 0" xyz="0.025 0.15 0.1875" />
-    <parent link="${robot_name_prop}_base_link" />
-    <child link="${robot_name_prop}_front_left_standoff" />
+    <parent link="chassis" />
+    <child link="front_left_standoff" />
   </joint>
   <!-- Back standoffs -->
-  <xacro:standoff name="${robot_name_prop}_back_right_standoff" />
-  <joint name="${robot_name_prop}_back_right_standoff_joint" type="fixed">
+  <xacro:standoff name="back_right_standoff" />
+  <joint name="back_right_standoff_joint" type="fixed">
     <origin rpy="0 0 0" xyz="-0.025 -0.15 0.1875" />
-    <parent link="${robot_name_prop}_base_link" />
-    <child link="${robot_name_prop}_back_right_standoff" />
-  </joint>
-  <xacro:standoff name="${robot_name_prop}_back_left_standoff" />
-  <joint name="${robot_name_prop}_back_left_standoff_joint" type="fixed">
+    <parent link="chassis" />
+    <child link="back_right_standoff" />
+  </joint>
+  <xacro:standoff name="back_left_standoff" />
+  <joint name="back_left_standoff_joint" type="fixed">
     <origin rpy="0 0 0" xyz="-0.025 0.15 0.1875" />
-    <parent link="${robot_name_prop}_base_link" />
-    <child link="${robot_name_prop}_back_left_standoff" />
+    <parent link="chassis" />
+    <child link="back_left_standoff" />
   </joint>
   <!-- Cup holder tray -->
-  <xacro:cup_holder_tray name="${robot_name_prop}_cup_holder" />
-  <joint name="${robot_name_prop}_cup_holder_joint" type="fixed">
+  <xacro:cup_holder_tray name="cup_holder" />
+  <joint name="cup_holder_joint" type="fixed">
     <origin rpy="0 0 0" xyz="0.0 0.0 0.3425" />
-    <parent link="${robot_name_prop}_base_link" />
-    <child link="${robot_name_prop}_cup_holder" />
-  </joint>
-  <gazebo reference="${robot_name_prop}_cup_holder">
+    <parent link="chassis" />
+    <child link="cup_holder" />
+  </joint>
+  <gazebo reference="cup_holder">
        <material>${chassis_material}</material>
   </gazebo>
   <!-- Wheel Left -->
-  <xacro:wheel prefix="${robot_name_prop}_left" />
-  <gazebo reference="${robot_name_prop}_left_wheel">
+  <xacro:wheel prefix="left" />
+  <gazebo reference="left_wheel">
     <kp>1000000000000000000000000000.0</kp>
     <kd>1000000000000000000000000000.0</kd>
-    <mu1>10.0</mu1>
-    <mu2>10.0</mu2>
+    <mu1>1.0</mu1>
+    <mu2>1.0</mu2>
     <material>Gazebo/Black</material>
   </gazebo>
-  <joint name="${robot_name_prop}_joint_left_wheel" type="continuous">
+  <joint name="joint_left_wheel" type="continuous">
     <origin rpy="0 0 0" xyz="0 0.12 -0.0775" />
-    <child link="${robot_name_prop}_left_wheel" />
-    <parent link="${robot_name_prop}_chassis" />
+    <child link="left_wheel" />
+    <parent link="chassis" />
     <axis rpy="0 0 0" xyz="0 1 0" />
     <limit effort="10000" velocity="1000" />
@@ -165,16 +167,16 @@
   </joint>
   <!-- Wheel Right -->
-  <xacro:wheel prefix="${robot_name_prop}_right" />
-  <gazebo reference="${robot_name_prop}_right_wheel">
+  <xacro:wheel prefix="right" />
+  <gazebo reference="right_wheel">
     <kp>1000000000000000000000000000.0</kp>
     <kd>1000000000000000000000000000.0</kd>
-    <mu1>10.0</mu1>
-    <mu2>10.0</mu2>
+    <mu1>1.0</mu1>
+    <mu2>1.0</mu2>
     <material>Gazebo/Black</material>
   </gazebo>
-  <joint name="${robot_name_prop}_joint_right_wheel" type="continuous">
+  <joint name="joint_right_wheel" type="continuous">
     <origin rpy="0 0 0" xyz="0 -0.12 -0.0775" />
-    <child link="${robot_name_prop}_right_wheel" />
-    <parent link="${robot_name_prop}_chassis" />
+    <child link="right_wheel" />
+    <parent link="chassis" />
     <axis rpy="0 0 0" xyz="0 1 0" />
     <limit effort="10000" velocity="1000" />
@@ -182,5 +184,5 @@
   </joint>
   <!-- Caster Wheel Front -->
-  <link name="${robot_name_prop}_front_yaw_link">
+  <link name="front_yaw_link">
     <visual>
       <origin rpy="0 1.5707 1.5707" xyz="0 0 0" />
@@ -202,16 +204,16 @@
     </inertial>
   </link>
-  <gazebo reference="${robot_name_prop}_front_yaw_link">
+  <gazebo reference="front_yaw_link">
         <material>Gazebo/Blue</material>
   </gazebo>
-  <joint name="${robot_name_prop}_front_yaw_joint" type="continuous">
+  <joint name="front_yaw_joint" type="continuous">
     <origin rpy="0 0 0" xyz="0.12 0 -0.1082" />
-    <parent link="${robot_name_prop}_chassis" />
-    <child link="${robot_name_prop}_front_yaw_link" />
+    <parent link="chassis" />
+    <child link="front_yaw_link" />
     <axis xyz="0 0 1" />
     <limit effort="1000.0" velocity="100.0" />
     <dynamics damping="0.0" friction="0.1" />
   </joint>
-  <link name="${robot_name_prop}_front_roll_link">
+  <link name="front_roll_link">
      <visual>
       <origin rpy="0 1.5707 1.5707" xyz="0 0 0" />
@@ -233,16 +235,16 @@
     </inertial>
   </link>
-  <gazebo reference="${robot_name_prop}_front_roll_link">
+  <gazebo reference="front_roll_link">
         <material>Gazebo/Red</material>
   </gazebo>
-  <joint name="${robot_name_prop}_front_roll_joint" type="continuous">
+  <joint name="front_roll_joint" type="continuous">
     <origin rpy="0 0 0" xyz="0 0 0" />
-    <parent link="${robot_name_prop}_front_yaw_link" />
-    <child link="${robot_name_prop}_front_roll_link" />
+    <parent link="front_yaw_link" />
+    <child link="front_roll_link" />
     <axis xyz="1 0 0" />
     <limit effort="1000.0" velocity="100.0" />
     <dynamics damping="0.0" friction="0.1" />
   </joint>
-  <link name="${robot_name_prop}_front_pitch_link">
+  <link name="front_pitch_link">
      <visual>
       <origin rpy="0 1.5707 1.5707" xyz="0 0 0" />
@@ -264,15 +266,15 @@
     </inertial>
   </link>
-  <gazebo reference="${robot_name_prop}_front_pitch_link">
+  <gazebo reference="front_pitch_link">
     <kp>1000000000000000000000000000.0</kp>
     <kd>1000000000000000000000000000.0</kd>
-    <mu1>0.5</mu1>
-    <mu2>0.5</mu2>
+    <mu1>0.001</mu1>
+    <mu2>0.001</mu2>
     <material>Gazebo/Purple</material>
   </gazebo>
-  <joint name="${robot_name_prop}_front_pitch_joint" type="continuous">
+  <joint name="front_pitch_joint" type="continuous">
     <origin rpy="0 0 0" xyz="0 0 0" />
-    <parent link="${robot_name_prop}_front_roll_link" />
-    <child link="${robot_name_prop}_front_pitch_link" />
+    <parent link="front_roll_link" />
+    <child link="front_pitch_link" />
     <axis xyz="0 1 0" />
     <limit effort="1000.0" velocity="100.0" />
@@ -280,5 +282,5 @@
   </joint>
   <!-- Caster Wheel Back -->
-  <link name="${robot_name_prop}_back_yaw_link">
+  <link name="back_yaw_link">
      <visual>
       <origin rpy="0 1.5707 1.5707" xyz="0 0 0" />
@@ -300,16 +302,16 @@
     </inertial>
   </link>
-  <gazebo reference="${robot_name_prop}_back_yaw_link">
+  <gazebo reference="back_yaw_link">
         <material>Gazebo/Blue</material>
   </gazebo>
-  <joint name="${robot_name_prop}_back_yaw_joint" type="continuous">
+  <joint name="back_yaw_joint" type="continuous">
     <origin rpy="0 0 0" xyz="-0.12 0 -0.1082" />
-    <parent link="${robot_name_prop}_chassis" />
-    <child link="${robot_name_prop}_back_yaw_link" />
+    <parent link="chassis" />
+    <child link="back_yaw_link" />
     <axis xyz="0 0 1" />
     <limit effort="1000.0" velocity="100.0" />
     <dynamics damping="0.0" friction="0.1" />
   </joint>
-  <link name="${robot_name_prop}_back_roll_link">
+  <link name="back_roll_link">
      <visual>
       <origin rpy="0 1.5707 1.5707" xyz="0 0 0" />
@@ -331,16 +333,16 @@
     </inertial>
   </link>
-  <gazebo reference="${robot_name_prop}_back_roll_link">
+  <gazebo reference="back_roll_link">
         <material>Gazebo/Red</material>
   </gazebo>
-  <joint name="${robot_name_prop}_back_roll_joint" type="continuous">
+  <joint name="back_roll_joint" type="continuous">
     <origin rpy="0 0 0" xyz="0 0 0" />
-    <parent link="${robot_name_prop}_back_yaw_link" />
-    <child link="${robot_name_prop}_back_roll_link" />
+    <parent link="back_yaw_link" />
+    <child link="back_roll_link" />
     <axis xyz="1 0 0" />
     <limit effort="1000.0" velocity="100.0" />
     <dynamics damping="0.0" friction="0.1" />
   </joint>
-  <link name="${robot_name_prop}_back_pitch_link">
+  <link name="back_pitch_link">
      <visual>
       <origin rpy="0 1.5707 1.5707" xyz="0 0 0" />
@@ -362,15 +364,15 @@
     </inertial>
   </link>
-  <gazebo reference="${robot_name_prop}_back_pitch_link">
+  <gazebo reference="back_pitch_link">
     <kp>1000000000000000000000000000.0</kp>
     <kd>1000000000000000000000000000.0</kd>
-    <mu1>0.5</mu1>
-    <mu2>0.5</mu2>
+    <mu1>0.001</mu1>
+    <mu2>0.001</mu2>
     <material>Gazebo/Yellow</material>
   </gazebo>
-  <joint name="${robot_name_prop}_back_pitch_joint" type="continuous">
+  <joint name="back_pitch_joint" type="continuous">
     <origin rpy="0 0 0" xyz="0 0 0" />
-    <parent link="${robot_name_prop}_back_roll_link" />
-    <child link="${robot_name_prop}_back_pitch_link" />
+    <parent link="back_roll_link" />
+    <child link="back_pitch_link" />
     <axis xyz="0 1 0" />
     <limit effort="1000.0" velocity="100.0" />
@@ -380,30 +382,31 @@
   <!-- JOINT PUBLISHER -->
   <gazebo>
-    <plugin name="${robot_name_prop}_robot_joint_state" filename="libgazebo_ros_joint_state_publisher.so">
+    <plugin name="robot_joint_state" filename="libgazebo_ros_joint_state_publisher.so">
       <ros>
-          <remapping>~/out:=/${robot_name_prop}/joint_states</remapping>
+            <namespace>${robot_name}</namespace>
+            <remapping>~/out:=/joint_states</remapping>
       </ros>
       <update_rate>30</update_rate>
-      <joint_name>${robot_name_prop}_joint_left_wheel</joint_name>
-      <joint_name>${robot_name_prop}_joint_right_wheel</joint_name>
-      <joint_name>${robot_name_prop}_front_yaw_joint</joint_name>
-      <joint_name>${robot_name_prop}_back_yaw_joint</joint_name>
-      <joint_name>${robot_name_prop}_front_roll_joint</joint_name>
-      <joint_name>${robot_name_prop}_back_roll_joint</joint_name>
-      <joint_name>${robot_name_prop}_front_pitch_joint</joint_name>
-      <joint_name>${robot_name_prop}_back_pitch_joint</joint_name>
+      <joint_name>joint_left_wheel</joint_name>
+      <joint_name>joint_right_wheel</joint_name>
+      <joint_name>front_yaw_joint</joint_name>
+      <joint_name>back_yaw_joint</joint_name>
+      <joint_name>front_roll_joint</joint_name>
+      <joint_name>back_roll_joint</joint_name>
+      <joint_name>front_pitch_joint</joint_name>
+      <joint_name>back_pitch_joint</joint_name>
     </plugin>
   </gazebo>
    <!-- Differential drive -->
   <gazebo>
-    <plugin filename="libgazebo_ros_diff_drive.so" name="${robot_name_prop}_differential_drive_controller">
-        <ros>
-          <!-- Remap default topics -->
-          <remapping>cmd_vel:=${robot_name_prop}/cmd_vel</remapping>
-          <remapping>odom:=${robot_name_prop}/odom</remapping>
-        </ros>
+    <plugin filename="libgazebo_ros_diff_drive.so" name="differential_drive_controller">
+      <!-- Topic to receive geometry_msgs/Twist message commands, defaults to `cmd_vel` -->
+      <ros>
+            <namespace>${robot_name}</namespace>
+            <remapping>~/cmd_vel:=cmd_vel</remapping>
+      </ros>
       <!-- wheels -->
-      <left_joint>${robot_name_prop}_joint_left_wheel</left_joint>
-      <right_joint>${robot_name_prop}_joint_right_wheel</right_joint>
+      <left_joint>joint_left_wheel</left_joint>
+      <right_joint>joint_right_wheel</right_joint>
       <!-- kinematics -->
       <wheel_separation>0.24</wheel_separation>
@@ -415,6 +418,6 @@
       <publish_odom>true</publish_odom>
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
File: xacro/cup_holder_tray.xacro (robot description, xacro)
@@ -9,5 +9,5 @@
           <cylinder length="${tray_length}" radius="${tray_radius}" />
         </geometry>
-        <material name="blue" />
+        <material name="rviz_material" />
       </visual>
       <collision>

Commit message: colors fixed

File: xacro/barista_robot_model.urdf.xacro (robot description, xacro)
@@ -10,15 +10,21 @@
 <xacro:arg name="robot_name" default="barista" />
 <xacro:property name="robot_name" value="$(arg robot_name)"/>
+<xacro:property name="robot_material" value="BlueMaterial"/>
+<material name="BlueMaterial">
+    <color rgba="0 0 1 1"/>
+</material>
+<material name="RedMaterial">
+    <color rgba="1 0 0 1"/>
+</material>
 <xacro:property name="chassis_material" value="Gazebo/Blue"/>
-<xacro:property name="rviz_chassis_material_blue" value="blue"/>
-<xacro:property name="rviz_chassis_material_red" value="red"/>
 <!-- Check if the robot is Rick and set color to Blue -->
 <xacro:if value="${robot_name == 'rick'}">
   <xacro:property name="chassis_material" value="Gazebo/Blue"/>
-  <xacro:property name="rviz_material" value="${rviz_chassis_material_blue}"/>
+  <xacro:property name="robot_material" value="BlueMaterial"/>
 </xacro:if>
 <!-- Check if the robot is Morty and set color to Red -->
 <xacro:if value="${robot_name == 'morty'}">
   <xacro:property name="chassis_material" value="Gazebo/Red"/>
+  <xacro:property name="robot_material" value="RedMaterial"/>
 </xacro:if>
 <!-- Lidar Sensor Macro Definition -->
@@ -92,5 +98,5 @@
         <cylinder length="0.155" radius="0.178" />
       </geometry>
-      <material name="rviz_material" />
+      <material name="${robot_material}" />
     </visual>
     <collision>

File: xacro/cup_holder_tray.xacro (robot description, xacro)
@@ -9,5 +9,5 @@
           <cylinder length="${tray_length}" radius="${tray_radius}" />
         </geometry>
-        <material name="rviz_material" />
+        <material name="${robot_material}" />
       </visual>
       <collision>

File: xacro/wheel.xacro (robot description, xacro)
@@ -10,4 +10,5 @@
                     <cylinder length="${wheel_width}" radius="${wheel_radius}" />
                 </geometry>
+                <material name="black" />
             </visual>
             <collision>

Commit message: gazebo lidar mesh issue fixed, laserscan rviz added, scan topic for each robot added

File: xacro/barista_robot_model.urdf.xacro (robot description, xacro)
@@ -30,22 +30,8 @@
 <!-- Lidar Sensor Macro Definition -->
 <xacro:macro name="laser_scanner">
-    <!-- Lidar Sensor -->
-    <link name="lidar">
-        <visual>
-            <origin rpy="0 0 0" xyz="0.0 0 -0.05" />
-            <geometry>
-                <mesh filename="package://barista_robot_description/meshes/hokuyo_urg_04lx.dae"/>
-            </geometry>
-        </visual>
-    </link>
-    <joint name="lidar_joint" type="fixed">
-        <origin rpy="0 0 0" xyz="-0.05 0 0.125" />
-        <parent link="chassis" />
-        <child link="lidar" />
-    </joint>
     <!-- Lidar plugin -->
     <gazebo reference="lidar">
         <material>Gazebo/Black</material>
-        <sensor name="sensor_ray" type="ray">
+        <sensor name="${robot_name}_sensor_ray" type="ray">
             <pose>0 0 0 0 0 0</pose>
             <ray>
@@ -66,8 +52,8 @@
             <visualize>true</visualize>
             <update_rate>100.0</update_rate>
-            <plugin name="laser" filename="libgazebo_ros_ray_sensor.so">
+            <plugin name="${robot_name}_laser" filename="libgazebo_ros_ray_sensor.so">
                 <ros>
                     <namespace>${robot_name}</namespace>
-                    <remapping>~/out:=/scan</remapping>
+                    <remapping>~/out:=/${robot_name}/scan</remapping>
                 </ros>
                 <frame_name>${robot_name}/base_link</frame_name>
@@ -119,4 +105,18 @@
       <material>${chassis_material}</material>
   </gazebo>
+      <!-- Lidar Sensor -->
+    <link name="lidar">
+        <visual>
+            <origin rpy="0 0 0" xyz="0.0 0 -0.05" />
+            <geometry>
+                <mesh filename="package://barista_robot_description/meshes/hokuyo_urg_04lx.dae"/>
+            </geometry>
+        </visual>
+    </link>
+    <joint name="lidar_joint" type="fixed">
+        <origin rpy="0 0 0" xyz="-0.05 0 0.125" />
+        <parent link="chassis" />
+        <child link="lidar" />
+    </joint>
   <!-- Front standoffs -->
   <xacro:standoff name="front_right_standoff" />
